File: metronome.sch (KiCad schematic (older format))
At the start: 11 parts, among them P1 CONN_01X02, U1 LM555N

Commit message: Revise circuit
Replace a 22uF capacitor in RC circuit to 4.7uF to get more usable range of frequency.
Parts:
- added SW1: SWITCH_INV, Connect:PINHEAD1-3, symbol SWITCH_INV
- C1: value 22uF -> 4.7uF
- RV1: footprint Potentiometers:Potentiometer_Alps-RK163-single_20mm -> Connect:PINHEAD1-3; symbol POT -> POT-RESCUE-metronome
Connections:
- net +9V: now also SW1.2; no longer P1.1 (P1)
- new net: P1.1 (P1), SW1.1
- no-connect marks 1 -> 2
Other:
- note added: "TODOs:\n- Add amplifier circuit to increase volume of speaker (with using a potential resistor to adjust volume)."
- note removed: "TODO: add an on/off switch here"
- moved on the sheet: P1
Changed lines of the file:
@@
 EESchema Schematic File Version 2
+LIBS:metronome-rescue
 LIBS:power
 LIBS:device
@@
 LIBS:contrib
 LIBS:valves
+LIBS:metronome-cache
 EELAYER 25 0
 EELAYER END
@@
 $EndComp
 $Comp
-L POT RV1
+L POT-RESCUE-metronome RV1
 U 1 1 57F36253
 P 4700 3350
 F 0 "RV1" H 4700 3250 50  0000 C CNN
 F 1 "POT" H 4700 3350 50  0000 C CNN
-F 2 "Potentiometers:Potentiometer_Alps-RK163-single_20mm" H 4700 3350 50  0001 C CNN
+F 2 "Connect:PINHEAD1-3" H 4700 3350 50  0001 C CNN
 F 3 "" H 4700 3350 50  0000 C CNN
 	1    4700 3350
@@
 P 3500 3400
 F 0 "C1" H 3525 3500 50  0000 L CNN
-F 1 "22uF" H 3525 3300 50  0000 L CNN
+F 1 "4.7uF" H 3525 3300 50  0000 L CNN
 F 2 "Discret:CP36V" H 3538 3250 50  0001 C CNN
 F 3 "" H 3500 3400 50  0000 C CNN
@@
 L +9V #PWR01
 U 1 1 57F364BD
-P 6300 1500
-F 0 "#PWR01" H 6300 1350 50  0001 C CNN
-F 1 "+9V" H 6300 1640 50  0000 C CNN
-F 2 "" H 6300 1500 50  0000 C CNN
-F 3 "" H 6300 1500 50  0000 C CNN
-	1    6300 1500
+P 7100 1400
+F 0 "#PWR01" H 7100 1250 50  0001 C CNN
+F 1 "+9V" H 7100 1540 50  0000 C CNN
+F 2 "" H 7100 1400 50  0000 C CNN
+F 3 "" H 7100 1400 50  0000 C CNN
+	1    7100 1400
 	1    0    0    -1
 $EndComp
@@
 L GND #PWR02
 U 1 1 57F364EF
-P 6300 1600
-F 0 "#PWR02" H 6300 1350 50  0001 C CNN
-F 1 "GND" H 6300 1450 50  0000 C CNN
-F 2 "" H 6300 1600 50  0000 C CNN
-F 3 "" H 6300 1600 50  0000 C CNN
-	1    6300 1600
+P 7100 1800
+F 0 "#PWR02" H 7100 1550 50  0001 C CNN
+F 1 "GND" H 7100 1650 50  0000 C CNN
+F 2 "" H 7100 1800 50  0000 C CNN
+F 3 "" H 7100 1800 50  0000 C CNN
+	1    7100 1800
 	1    0    0    -1
 $EndComp
@@
 L CONN_01X02 P1
 U 1 1 57F36517
-P 6750 1550
-F 0 "P1" H 6750 1700 50  0000 C CNN
-F 1 "CONN_01X02" V 6850 1550 50  0000 C CNN
-F 2 "Pin_Headers:Pin_Header_Angled_1x02" H 6750 1550 50  0001 C CNN
-F 3 "" H 6750 1550 50  0000 C CNN
-	1    6750 1550
+P 8650 1500
+F 0 "P1" H 8650 1650 50  0000 C CNN
+F 1 "CONN_01X02" V 8750 1500 50  0000 C CNN
+F 2 "Pin_Headers:Pin_Header_Angled_1x02" H 8650 1500 50  0001 C CNN
+F 3 "" H 8650 1500 50  0000 C CNN
+	1    8650 1500
 	1    0    0    -1
 $EndComp
 NoConn ~ 3600 2500
-Wire Wire Line
-	6550 1500 6300 1500
-Wire Wire Line
-	6550 1600 6300 1600
 Wire Wire Line
 	3600 2700 3500 2700
@@
 Wire Wire Line
 	4700 1850 4700 1650
-Wire Wire Line
-	4700 1650 5350 1650
 Connection ~ 5200 1650
 Wire Wire Line
@@
 $Comp
 L PWR_FLAG #FLG08
-U 1 1 57F372EB
-P 6500 1650
-F 0 "#FLG08" H 6500 1745 50  0001 C CNN
-F 1 "PWR_FLAG" H 6500 1830 50  0000 C CNN
-F 2 "" H 6500 1650 50  0000 C CNN
-F 3 "" H 6500 1650 50  0000 C CNN
-	1    6500 1650
-	-1   0    0    1
-$EndComp
-$Comp
-L PWR_FLAG #FLG09
 U 1 1 57F37315
-P 5350 1650
-F 0 "#FLG09" H 5350 1745 50  0001 C CNN
-F 1 "PWR_FLAG" H 5350 1830 50  0000 C CNN
-F 2 "" H 5350 1650 50  0000 C CNN
-F 3 "" H 5350 1650 50  0000 C CNN
-	1    5350 1650
-	0    1    1    0
-$EndComp
-Wire Wire Line
-	6500 1650 6500 1600
-Connection ~ 6500 1600
-$Comp
-L GND #PWR010
+P 6850 1550
+F 0 "#FLG08" H 6850 1645 50  0001 C CNN
+F 1 "PWR_FLAG" H 6850 1730 50  0000 C CNN
+F 2 "" H 6850 1550 50  0000 C CNN
+F 3 "" H 6850 1550 50  0000 C CNN
+	1    6850 1550
+	0    -1   -1   0
+$EndComp
+$Comp
+L GND #PWR09
 U 1 1 57F374D7
 P 4100 1950
-F 0 "#PWR010" H 4100 1700 50  0001 C CNN
+F 0 "#PWR09" H 4100 1700 50  0001 C CNN
 F 1 "GND" H 4100 1800 50  0000 C CNN
 F 2 "" H 4100 1950 50  0000 C CNN
@@
 $EndComp
 $Comp
-L +9V #PWR011
+L +9V #PWR010
 U 1 1 57F37501
 P 4100 3150
-F 0 "#PWR011" H 4100 3000 50  0001 C CNN
+F 0 "#PWR010" H 4100 3000 50  0001 C CNN
 F 1 "+9V" H 4100 3290 50  0000 C CNN
 F 2 "" H 4100 3150 50  0000 C CNN
@@
 Wire Wire Line
 	4100 3150 4100 2900
-Text Notes 6050 1200 0    60   ~ 0
-TODO: add an on/off switch here
+$Comp
+L SWITCH_INV SW1
+U 1 1 57F3DA9F
+P 7600 1550
+F 0 "SW1" H 7400 1700 50  0000 C CNN
+F 1 "SWITCH_INV" H 7450 1400 50  0000 C CNN
+F 2 "Connect:PINHEAD1-3" H 7600 1550 50  0001 C CNN
+F 3 "" H 7600 1550 50  0000 C CNN
+	1    7600 1550
+	1    0    0    -1
+$EndComp
+Wire Wire Line
+	7100 1550 7100 1400
+Wire Wire Line
+	8450 1450 8100 1450
+Wire Wire Line
+	8450 1550 8250 1550
+Wire Wire Line
+	8250 1550 8250 1800
+Wire Wire Line
+	8250 1800 7100 1800
+NoConn ~ 8100 1650
+$Comp
+L PWR_FLAG #FLG011
+U 1 1 57F3DD22
+P 7900 1950
+F 0 "#FLG011" H 7900 2045 50  0001 C CNN
+F 1 "PWR_FLAG" H 7900 2130 50  0000 C CNN
+F 2 "" H 7900 1950 50  0000 C CNN
+F 3 "" H 7900 1950 50  0000 C CNN
+	1    7900 1950
+	-1   0    0    1
+$EndComp
+Wire Wire Line
+	7900 1950 7900 1800
+Connection ~ 7900 1800
+Wire Wire Line
+	6850 1550 7100 1550
+Wire Wire Line
+	4700 1650 5200 1650
+Text Notes 5250 4700 0    60   ~ 0
+TODOs:\n- Add amplifier circuit to increase volume of speaker (with using a potential resistor to adjust volume).
 $EndSCHEMATC
